Commit message: Clean up code

File: NUgus.urdf (robot description, URDF)
Before this commit: robot nubots_nugus_hull, 21 links, 20 joints
Joints:
- joint left_ankle_pitch: axis -1  0  0 -> 0 -1  0; origin xyz=0    0.01 -0.2 rpy=3.14159  0      -3.14159 -> xyz=0 0 -0.2 rpy=0 0 0
- joint left_ankle_roll: axis 0 -1  0 -> 1 0 0; origin xyz=0    0.04  0 rpy=-3.14159  0      -3.14159 -> xyz=-0.04 0 0 rpy=0 0 0
- joint left_hip_pitch: axis 1  0  0 -> 0 -1 0; origin xyz=0   -0.01  0 rpy=-0.05  0    0 -> xyz=0.01 0 0.01 rpy=0 0 0
- joint left_hip_roll: axis 0 -1  0 -> 1 0 0
- joint left_hip_yaw: origin xyz=0     0.055  0 rpy=0       0       1.57079 -> xyz=0 0.055 0 rpy=0 0 0
- joint left_knee_pitch: axis 1  0  0 -> 0 -1  0; origin xyz=0       0.00949 -0.18976 rpy=0.05  0    0 -> xyz=0 0 -0.2 rpy=0 0 0
- joint right_ankle_pitch: axis -1  0  0 -> 0 1 0; origin xyz=0    0.01 -0.2 rpy=3.14159  0      -3.14159 -> xyz=0 0 -0.2 rpy= 0 0 0
- joint right_ankle_roll: axis 0 -1  0 -> 1 0 0; origin xyz=0    0.04  0 rpy=-3.14159  0      -3.14159 -> xyz=-0.04 0 0 rpy=0 0 0
- joint right_hip_pitch: axis 1  0  0 -> 0 1 0; origin xyz=0   -0.01  0.01 rpy=-0.05  0    0 -> xyz=0.01 0 0.01 rpy=0 0 0
- joint right_hip_roll: axis 0 -1  0 -> 1 0 0
- joint right_hip_yaw: origin xyz=0    -0.055  0 rpy=0       0       1.57079 -> xyz=0    -0.055  0 rpy=0 0 0
- joint right_knee_pitch: axis 1  0  0 -> 0 1 0; origin xyz=0       0.00999 -0.19975 rpy=0.05  0    0 -> xyz=0 0 -0.2 rpy=0 0 0

Commit message: Implement quasi-static routine

File: NUgus.urdf (robot description, URDF)
Before this commit: robot nubots_nugus_hull, 21 links, 20 joints
Joints:
- joint left_ankle_pitch: axis 0 -1  0 -> 0 1  0
- joint left_hip_pitch: axis 0 -1 0 -> 0 1 0
- joint left_knee_pitch: axis 0 -1  0 -> 0 1  0

Commit message: Tune gait parameters

File: NUgus.urdf (robot description, URDF)
Before this commit: robot nubots_nugus_hull, 21 links, 20 joints
Joints:
- joint left_ankle_roll: origin xyz=-0.04 0 0 rpy=0 0 0 -> xyz=0 0 0 rpy=0 0 0
- joint left_hip_pitch: origin xyz=0.01 0 0.01 rpy=0 0 0 -> xyz=0 0 0 rpy=0 0 0
- joint right_ankle_roll: origin xyz=-0.04 0 0 rpy=0 0 0 -> xyz=0 0 0 rpy=0 0 0
- joint right_hip_pitch: origin xyz=0.01 0 0.01 rpy=0 0 0 -> xyz=0 0 0 rpy=0 0 0

Commit message: Add CoM calculations
Currently not sure on these

File: NUgus.urdf (robot description, URDF)
Before this commit: robot nubots_nugus_hull, 21 links, 20 joints
Links:
- link head: mass 0.419 -> 0
- link left_lower_arm: mass 0.26 -> 0
- link left_shoulder: mass 0.025434 -> 0
- link left_upper_arm: mass 0.297 -> 0
- link neck: mass 0.135 -> 0
- link right_lower_arm: mass 0.26 -> 0
- link right_shoulder: mass 0.025434 -> 0
- link right_upper_arm: mass 0.297 -> 0
- link torso: mass 2.539 -> 4.2530

Commit message: Optimize Kinematics

File: NUgus.urdf (robot description, URDF)
Before this commit: robot nubots_nugus_hull, 21 links, 20 joints
Links:
- link head: mass 0 -> 4.2530
- link torso: mass 4.2530 -> 0
