Commit message: Add new urdf

File: robot.urdf (robot description, URDF)
Before this commit: robot onshape, 21 links, 20 joints
Links:
- removed link right_lower_arm
- added link left_lower_arm_copy_1, mass 0.357122; collision mesh filename=meshes/left_lower_arm_copy_1_collision.stl; visual mesh filename=meshes/left_lower_arm_copy_1_visual.stl
- link head: geometry collision mesh filename=meshes/head_collision.stl; visual mesh filename=meshes/head_visual.stl
- link left_ankle: mass 0.395953 -> 0.329993; geometry collision mesh filename=meshes/left_ankle_collision.stl; visual mesh filename=meshes/left_ankle_visual.stl
- link left_ankle_2: mass 0.395953 -> 0.329993; geometry collision mesh filename=meshes/left_ankle_2_collision.stl; visual mesh filename=meshes/left_ankle_2_visual.stl
- link left_foot: geometry collision mesh filename=meshes/left_foot_collision.stl; visual mesh filename=meshes/left_foot_visual.stl
- link left_hip_roll: geometry collision mesh filename=meshes/left_hip_roll_collision.stl; visual mesh filename=meshes/left_hip_roll_visual.stl
- link left_hip_yaw: geometry collision mesh filename=meshes/left_hip_yaw_collision.stl; visual mesh filename=meshes/left_hip_yaw_visual.stl
- link left_lower_arm: geometry collision mesh filename=meshes/left_lower_arm_collision.stl; visual mesh filename=meshes/left_lower_arm_visual.stl
- link left_shoulder: geometry collision mesh filename=meshes/left_shoulder_collision.stl; visual mesh filename=meshes/left_shoulder_visual.stl
- link left_upper_arm: geometry collision mesh filename=meshes/left_upper_arm_collision.stl; visual mesh filename=meshes/left_upper_arm_visual.stl
- link left_upper_leg: mass 0 -> 1.24036; geometry collision mesh filename=meshes/left_upper_leg_collision.stl; visual mesh filename=meshes/left_upper_leg_visual.stl
- link lower_leg_left: geometry collision mesh filename=meshes/lower_leg_left_collision.stl; visual mesh filename=meshes/lower_leg_left_visual.stl
- link lower_leg_right: geometry collision mesh filename=meshes/lower_leg_right_collision.stl; visual mesh filename=meshes/lower_leg_right_visual.stl
- link neck: mass 0.164974 -> 0.16501; geometry collision mesh filename=meshes/neck_collision.stl; visual mesh filename=meshes/neck_visual.stl
- link right_foot: geometry collision mesh filename=meshes/right_foot_collision.stl; visual mesh filename=meshes/right_foot_visual.stl
- link right_hip_roll: geometry collision mesh filename=meshes/right_hip_roll_collision.stl; visual mesh filename=meshes/right_hip_roll_visual.stl
- link right_hip_yaw: geometry collision mesh filename=meshes/right_hip_yaw_collision.stl; visual mesh filename=meshes/right_hip_yaw_visual.stl
- link right_shoulder: geometry collision mesh filename=meshes/right_shoulder_collision.stl; visual mesh filename=meshes/right_shoulder_visual.stl
- link right_upper_arm: geometry collision mesh filename=meshes/right_upper_arm_collision.stl; visual mesh filename=meshes/right_upper_arm_visual.stl
- link right_upper_leg: mass 0 -> 1.24036; geometry collision mesh filename=meshes/right_upper_leg_collision.stl; visual mesh filename=meshes/right_upper_leg_visual.stl
- link torso: mass 1.73566 -> 2.1698; geometry collision mesh filename=meshes/torso_collision.stl; visual mesh filename=meshes/torso_visual.stl
Joints:
- removed joint left_shoulder_pitch [shoulder]
- removed joint right_shoulder_pitch [shoulder]
- added joint left_shoulder_pitch: type revolute, parent torso, child left_shoulder, origin xyz=3.99598e-16 0.077 0.17775 rpy=-1.5708 5.16765e-16 -1.83187e-15, axis 0 0 1, limit effort=1 velocity=20
- added joint right_shoulder_pitch: type revolute, parent torso, child right_shoulder, origin xyz=1.17933e-16 -0.077 0.17775 rpy=-1.5708 4.4981e-16 -1.83187e-15, axis 0 0 1, limit effort=1 velocity=20
- joint left_ankle_pitch: origin xyz=0.199419 -0.00566882 -0.0002 rpy=-7.89113e-15 3.33307e-14 -5.36082e-15 -> xyz=0.199419 -0.00566882 -0.0002 rpy=-2.21654e-15 1.5961e-15 2.03982e-19
- joint left_ankle_roll: origin xyz=-7.77156e-16 -6.94565e-06 -0.000982442 rpy=1.5708 -1.73595e-13 1.20642e-14 -> xyz=-1.66533e-15 -6.94565e-06 -0.000982442 rpy=1.5708 -8.69144e-15 7.83425e-14
- joint left_elbow_pitch: child left_lower_arm -> left_lower_arm_copy_1; origin xyz=0.1575 -0.0235 0.0033 rpy=-1.5708 -9.71445e-16 -6.48574e-17 -> xyz=0.1575 -4.16334e-16 0.0033 rpy=-1.5708 -1.19349e-15 1.56366e-15
- joint left_hip_pitch: origin xyz=-2.2482e-15 2.9564e-05 0.06895 rpy=-1.5708 1.38608e-12 1.27676e-15 -> xyz=-2.30371e-15 2.9564e-05 0.06895 rpy=-1.5708 1.38608e-12 1.27676e-15
- joint left_knee_pitch: origin xyz=0.199541 -2.33261e-05 -0.0015 rpy=1.49726e-16 -6.55433e-14 -0.00523599 -> xyz=0.199541 -2.33261e-05 -0.00095424 rpy=-2.65601e-14 -5.52844e-14 -3.59878e-05
- joint right_ankle_pitch: origin xyz=0.199419 -0.00566882 0.0015 rpy=-6.49294e-16 6.91322e-16 -1.74705e-14 -> xyz=0.199419 -0.00566882 0.0015 rpy=-1.28717e-16 6.42564e-16 -1.12766e-16
- joint right_ankle_roll: origin xyz=-2.16493e-15 -6.94565e-06 -0.000982442 rpy=1.5708 -1.17408e-13 2.60917e-14 -> xyz=-2.22045e-15 -0.000116046 -0.000982442 rpy=1.5708 -1.1811e-13 2.53365e-14
- joint right_elbow_pitch: child right_lower_arm -> left_lower_arm; origin xyz=0.155337 0.023814 0.00263175 rpy=-1.5708 1.5708 0 -> xyz=0.157491 0.000314045 0.00263175 rpy=-1.5708 1.18239e-14 2.57201e-14
- joint right_knee_pitch: origin xyz=0.199541 -2.33261e-05 -0.0015 rpy=-2.76263e-14 -5.50623e-14 -0.00523599 -> xyz=0.199541 -2.33261e-05 -0.0015 rpy=-2.84504e-14 -5.46771e-14 6.40122e-05
